Commit message: update mass and motor model

File: resources/robots/dragon/dragon.urdf (robot description, URDF)
Before this commit: robot multirotor, 10 links, 9 joints
Links:
- link base_link: mass 0.40220 -> 0.665

Commit message: fix motor locations

File: resources/robots/dragon/dragon.urdf (robot description, URDF)
Before this commit: robot multirotor, 10 links, 9 joints
Joints:
- joint base_link_to_arm_motor_1: origin xyz=-0.036315 -0.04328 0.0 rpy=1.5707963267948968 2.220446049250313e-16 -0.7853981633974482 -> xyz=-0.036315 0.04328 0.0 rpy=1.5707963267948968 0.0 -2.3561944901923453
- joint base_link_to_arm_motor_2: origin xyz=-0.036315 0.04328 0.0 rpy=1.5707963267948968 0.0 -2.3561944901923453 -> xyz=0.036315 0.04328 0.0 rpy=-1.5707963267948968 0.0 -0.7853981633974482
- joint base_link_to_arm_motor_3: origin xyz=0.036315 0.04328 0.0 rpy=-1.5707963267948968 0.0 -0.7853981633974482 -> xyz=-0.036315 -0.04328 0.0 rpy=1.5707963267948968 2.220446049250313e-16 -0.7853981633974482
- joint base_link_to_motor_1: origin xyz=-0.07263 -0.08656 0.0 rpy=0.0 0.0 0.0 -> xyz=-0.07263 0.08656 0.0 rpy=0.0 0.0 0.0
- joint base_link_to_motor_2: origin xyz=-0.07263 0.08656 0.0 rpy=0.0 0.0 0.0 -> xyz=0.07263 0.08656 0.0 rpy=0.0 0.0 0.0
- joint base_link_to_motor_3: origin xyz=0.07263 0.08656 0.0 rpy=0.0 0.0 0.0 -> xyz=-0.07263 -0.08656 0.0 rpy=0.0 0.0 0.0

Commit message: improve dragon  model

File: resources/robots/dragon/dragon.urdf (robot description, URDF)
Before this commit: robot multirotor, 10 links, 9 joints
Links:
- link base_link: mass 0.665 -> 0.703
- link motor_0: mass 0.03307 -> 0.000001
- link motor_1: mass 0.03307 -> 0.000001
- link motor_2: mass 0.03307 -> 0.000001
- link motor_3: mass 0.03307 -> 0.000001
